Commit message: added rviz materials

File: rvbot_description/urdf/materials.xacro (robot description, xacro)
@@ -1,6 +1,15 @@
 <?xml version="1.0" ?>
 <robot name="rvbot" xmlns:xacro="http://www.ros.org/wiki/xacro" >
-<material name="silver">
-  <color rgba="0.700 0.700 0.700 1.000"/>
+<material name="white">
+  <color rgba="1.000 1.000 1.000 1.000"/>
+</material>
+<material name="black">
+  <color rgba="0.000 0.000 0.000 1.000"/>
+</material>
+<material name="blue">
+  <color rgba="0.000 0.000 1.000 1.000"/>
+</material>
+<material name="grey">
+  <color rgba="0.500 0.500 0.500 1.000"/>
 </material>
 </robot>

File: rvbot_description/urdf/rvbot.xacro (robot description, xacro)
@@ -17,5 +17,5 @@
       <mesh filename="package://rvbot_description/meshes/base_link.stl" scale="0.001 0.001 0.001"/>
     </geometry>
-    <material name="silver"/>
+    <material name="white"/>
   </visual>
   <collision>
@@ -37,5 +37,5 @@
       <mesh filename="package://rvbot_description/meshes/wheel_right.stl" scale="0.001 0.001 0.001"/>
     </geometry>
-    <material name="silver"/>
+    <material name="black"/>
   </visual>
   <collision>
@@ -57,5 +57,5 @@
       <mesh filename="package://rvbot_description/meshes/wheel_left.stl" scale="0.001 0.001 0.001"/>
     </geometry>
-    <material name="silver"/>
+    <material name="black"/>
   </visual>
   <collision>
@@ -77,5 +77,5 @@
       <mesh filename="package://rvbot_description/meshes/caster_front.stl" scale="0.001 0.001 0.001"/>
     </geometry>
-    <material name="silver"/>
+    <material name="grey"/>
   </visual>
   <collision>
@@ -97,5 +97,5 @@
       <mesh filename="package://rvbot_description/meshes/caster_back.stl" scale="0.001 0.001 0.001"/>
     </geometry>
-    <material name="silver"/>
+    <material name="grey"/>
   </visual>
   <collision>
@@ -117,5 +117,5 @@
       <mesh filename="package://rvbot_description/meshes/lidar_bottom.stl" scale="0.001 0.001 0.001"/>
     </geometry>
-    <material name="silver"/>
+    <material name="blue"/>
   </visual>
   <collision>
@@ -137,5 +137,5 @@
       <mesh filename="package://rvbot_description/meshes/lidar_top.stl" scale="0.001 0.001 0.001"/>
     </geometry>
-    <material name="silver"/>
+    <material name="blue"/>
   </visual>
   <collision>
