Commit message: removed _1

File: rvbot_description/urdf/rvbot.xacro (robot description, xacro)
@@ -24,5 +24,5 @@
   </collision>
 </link>
-<link name="wheel_right_1">
+<link name="wheel_right">
   <inertial>
     <origin rpy="0 0 0" xyz="1.2983705934591556e-17 -0.02930159298956944 -2.0539927481078024e-07"/>
@@ -33,5 +33,5 @@
     <origin rpy="0 0 0" xyz="-0.0 0.14 -0.061983"/>
     <geometry>
-      <mesh filename="package://rvbot_description/meshes/wheel_right_1.stl" scale="0.001 0.001 0.001"/>
+      <mesh filename="package://rvbot_description/meshes/wheel_right.stl" scale="0.001 0.001 0.001"/>
     </geometry>
     <material name="silver"/>
@@ -40,9 +40,9 @@
     <origin rpy="0 0 0" xyz="-0.0 0.14 -0.061983"/>
     <geometry>
-      <mesh filename="package://rvbot_description/meshes/wheel_right_1.stl" scale="0.001 0.001 0.001"/>
+      <mesh filename="package://rvbot_description/meshes/wheel_right.stl" scale="0.001 0.001 0.001"/>
     </geometry>
   </collision>
 </link>
-<link name="wheel_left_1">
+<link name="wheel_left">
   <inertial>
     <origin rpy="0 0 0" xyz="1.2983705934591556e-17 0.02930159298956947 -2.0539927483159692e-07"/>
@@ -53,5 +53,5 @@
     <origin rpy="0 0 0" xyz="-0.0 -0.14 -0.061983"/>
     <geometry>
-      <mesh filename="package://rvbot_description/meshes/wheel_left_1.stl" scale="0.001 0.001 0.001"/>
+      <mesh filename="package://rvbot_description/meshes/wheel_left.stl" scale="0.001 0.001 0.001"/>
     </geometry>
     <material name="silver"/>
@@ -60,9 +60,9 @@
     <origin rpy="0 0 0" xyz="-0.0 -0.14 -0.061983"/>
     <geometry>
-      <mesh filename="package://rvbot_description/meshes/wheel_left_1.stl" scale="0.001 0.001 0.001"/>
+      <mesh filename="package://rvbot_description/meshes/wheel_left.stl" scale="0.001 0.001 0.001"/>
     </geometry>
   </collision>
 </link>
-<link name="caster_front_1">
+<link name="caster_front">
   <inertial>
     <origin rpy="0 0 0" xyz="0.1 0.0 -0.02052622199592666"/>
@@ -73,5 +73,5 @@
     <origin rpy="0 0 0" xyz="-0.0 -0.0 -0.04425"/>
     <geometry>
-      <mesh filename="package://rvbot_description/meshes/caster_front_1.stl" scale="0.001 0.001 0.001"/>
+      <mesh filename="package://rvbot_description/meshes/caster_front.stl" scale="0.001 0.001 0.001"/>
     </geometry>
     <material name="silver"/>
@@ -80,9 +80,9 @@
     <origin rpy="0 0 0" xyz="-0.0 -0.0 -0.04425"/>
     <geometry>
-      <mesh filename="package://rvbot_description/meshes/caster_front_1.stl" scale="0.001 0.001 0.001"/>
+      <mesh filename="package://rvbot_description/meshes/caster_front.stl" scale="0.001 0.001 0.001"/>
     </geometry>
   </collision>
 </link>
-<link name="caster_back_1">
+<link name="caster_back">
   <inertial>
     <origin rpy="0 0 0" xyz="-0.10000000000000002 0.0 -0.02052622199592667"/>
@@ -93,5 +93,5 @@
     <origin rpy="0 0 0" xyz="-0.0 -0.0 -0.04425"/>
     <geometry>
-      <mesh filename="package://rvbot_description/meshes/caster_back_1.stl" scale="0.001 0.001 0.001"/>
+      <mesh filename="package://rvbot_description/meshes/caster_back.stl" scale="0.001 0.001 0.001"/>
     </geometry>
     <material name="silver"/>
@@ -100,9 +100,9 @@
     <origin rpy="0 0 0" xyz="-0.0 -0.0 -0.04425"/>
     <geometry>
-      <mesh filename="package://rvbot_description/meshes/caster_back_1.stl" scale="0.001 0.001 0.001"/>
+      <mesh filename="package://rvbot_description/meshes/caster_back.stl" scale="0.001 0.001 0.001"/>
     </geometry>
   </collision>
 </link>
-<link name="lidar_bottom_1">
+<link name="lidar_bottom">
   <inertial>
     <origin rpy="0 0 0" xyz="0.011999996295019591 -4.7482720637347705e-07 0.004999999999999977"/>
@@ -113,5 +113,5 @@
     <origin rpy="0 0 0" xyz="-0.023994 -0.000583 -0.23675"/>
     <geometry>
-      <mesh filename="package://rvbot_description/meshes/lidar_bottom_1.stl" scale="0.001 0.001 0.001"/>
+      <mesh filename="package://rvbot_description/meshes/lidar_bottom.stl" scale="0.001 0.001 0.001"/>
     </geometry>
     <material name="silver"/>
@@ -120,9 +120,9 @@
     <origin rpy="0 0 0" xyz="-0.023994 -0.000583 -0.23675"/>
     <geometry>
-      <mesh filename="package://rvbot_description/meshes/lidar_bottom_1.stl" scale="0.001 0.001 0.001"/>
+      <mesh filename="package://rvbot_description/meshes/lidar_bottom.stl" scale="0.001 0.001 0.001"/>
     </geometry>
   </collision>
 </link>
-<link name="lidar_top_1">
+<link name="lidar_top">
   <inertial>
     <origin rpy="0 0 0" xyz="-3.704980405805358e-09 -4.7482720637456125e-07 0.005000000000000032"/>
@@ -133,5 +133,5 @@
     <origin rpy="0 0 0" xyz="-0.035994 -0.000583 -0.24675"/>
     <geometry>
-      <mesh filename="package://rvbot_description/meshes/lidar_top_1.stl" scale="0.001 0.001 0.001"/>
+      <mesh filename="package://rvbot_description/meshes/lidar_top.stl" scale="0.001 0.001 0.001"/>
     </geometry>
     <material name="silver"/>
@@ -140,5 +140,5 @@
     <origin rpy="0 0 0" xyz="-0.035994 -0.000583 -0.24675"/>
     <geometry>
-      <mesh filename="package://rvbot_description/meshes/lidar_top_1.stl" scale="0.001 0.001 0.001"/>
+      <mesh filename="package://rvbot_description/meshes/lidar_top.stl" scale="0.001 0.001 0.001"/>
     </geometry>
   </collision>
@@ -147,5 +147,5 @@
   <origin rpy="0 0 0" xyz="0.0 -0.14 0.061983"/>
   <parent link="base_link"/>
-  <child link="wheel_right_1"/>
+  <child link="wheel_right"/>
   <axis xyz="0.0 -1.0 0.0"/>
 </joint>
@@ -153,5 +153,5 @@
   <origin rpy="0 0 0" xyz="0.0 0.14 0.061983"/>
   <parent link="base_link"/>
-  <child link="wheel_left_1"/>
+  <child link="wheel_left"/>
   <axis xyz="0.0 1.0 0.0"/>
 </joint>
@@ -159,20 +159,20 @@
   <origin rpy="0 0 0" xyz="0.0 0.0 0.04425"/>
   <parent link="base_link"/>
-  <child link="caster_front_1"/>
+  <child link="caster_front"/>
 </joint>
 <joint name="Rigid4" type="fixed">
   <origin rpy="0 0 0" xyz="0.0 0.0 0.04425"/>
   <parent link="base_link"/>
-  <child link="caster_back_1"/>
+  <child link="caster_back"/>
 </joint>
 <joint name="lidar_joint_bottom" type="fixed">
   <origin rpy="0 0 0" xyz="0.023994 0.000583 0.23675"/>
   <parent link="base_link"/>
-  <child link="lidar_bottom_1"/>
+  <child link="lidar_bottom"/>
 </joint>
 <joint name="lidar_joint_top" type="fixed">
   <origin rpy="0 0 0" xyz="0.012 0.0 0.01"/>
-  <parent link="lidar_bottom_1"/>
-  <child link="lidar_top_1"/>
+  <parent link="lidar_bottom"/>
+  <child link="lidar_top"/>
 </joint>
 </robot>

Commit message: Robot Manual Control

File: rvbot_description/urdf/rvbot.xacro (robot description, xacro)
@@ -3,5 +3,7 @@
 <xacro:include filename="$(find rvbot_description)/urdf/materials.xacro" />
 <xacro:include filename="$(find rvbot_description)/urdf/rvbot.trans" />
-<xacro:include filename="$(find rvbot_description)/urdf/rvbot.gazebo" />
+<xacro:include filename="$(find rvbot_description)/gazebo/rvbot_materials.gazebo" />
+<xacro:include filename="$(find rvbot_description)/gazebo/rvbot_physics.gazebo" />
+<xacro:include filename="$(find rvbot_description)/gazebo/rvbot_plugins.gazebo" />
 <link name="base_link">
   <inertial>
@@ -148,5 +150,5 @@
   <parent link="base_link"/>
   <child link="wheel_right"/>
-  <axis xyz="0.0 -1.0 0.0"/>
+  <axis xyz="0.0 1.0 0.0"/>
 </joint>
 <joint name="motor_left" type="continuous">

Commit message: lidar fixed

File: rvbot_description/urdf/rvbot.xacro (robot description, xacro)
@@ -174,5 +174,5 @@
 </joint>
 <joint name="lidar_joint_top" type="fixed">
-  <origin rpy="0 0 0" xyz="0.012 0.0 0.01"/>
+  <origin rpy="0 0 3.14159" xyz="0.012 0.0 0.01"/>
   <parent link="lidar_bottom"/>
   <child link="lidar_top"/>
